File: PCB/PCFanController.kicad_sch (KiCad schematic)
At the start: 19 parts, among them J1 USB_C_Receptacle_USB2.0_16P, M1 Fan_4pin, Q1 BSS138, U1 74HC595, U2 ATtiny404-SS, U3 74HC595, U4 CH221K, U5 AZ1117-3.3

Commit message: .
Parts:
- removed U5: AZ1117-3.3, Package_TO_SOT_SMD:SOT-223-3_TabPin2, symbol Regulator_Linear:AZ1117-3.3
- added C2: 10u, Capacitor_SMD:C_0603_1608Metric, symbol Device:C
- added C3: 0.1u, Capacitor_SMD:C_0603_1608Metric, symbol Device:C
- added C4: 22u, Capacitor_SMD:C_0603_1608Metric, symbol Device:C
- added C5: 47p, Capacitor_SMD:C_0603_1608Metric, symbol Device:C
- added C6: C, Capacitor_SMD:C_0603_1608Metric, symbol Device:C
- added L1: 1.2u, symbol Device:L
- added R11: 100k, Resistor_SMD:R_0603_1608Metric, symbol Device:R
- added R12: 30k, Resistor_SMD:R_0603_1608Metric, symbol Device:R
- added R13: 135k, Resistor_SMD:R_0603_1608Metric, symbol Device:R
- added SW1, SW2, SW3: SW_Push, symbol Switch:SW_Push
- added U5: OSL40562-LR, Display_7Segment:CA56-12EWA, symbol Display_Character:CC56-12EWA
- added U6: PTPS561243DRLR, footprints:DRL0006A-MFG, symbol lib:PTPS561243DRLR
- C1: footprint (none) -> Capacitor_SMD:C_0603_1608Metric
- R1, R2, R3, R4, R5, R6, R7, R8: value R -> 47; footprint (none) -> Resistor_SMD:R_0603_1608Metric
- R10, R9: footprint Package_TO_SOT_SMD:SOT-23-6 -> Resistor_SMD:R_0603_1608Metric
- U1, U3: footprint (none) -> Package_SO:TSSOP-16_4.4x5mm_P0.65mm
Connections:
- net +3V3: now also C4.2, C5.2, C6.2, L1.2, R13.1
- net 7seg-0: now also U5.6 (CC4)
- net 7seg-1: now also U5.8 (CC3)
- net 7seg-2: now also U5.9 (CC2)
- net 7seg-3: now also U5.12 (CC1)
- net 7seg-A: now also U5.11 (a)
- net 7seg-B: now also U5.7 (b)
- net 7seg-C: now also U5.4 (c)
- net 7seg-D: now also U5.2 (d)
- net 7seg-E: now also U5.1 (e)
- net 7seg-F: now also U5.10 (f)
- net 7seg-G: now also U5.5 (g)
- net 7seg-P: now also U5.3 (DPX)
- net Ctrl-A: now also SW1.1
- net Ctrl-B: now also SW2.1
- net Ctrl-Push: now also SW3.1
- net GND: now also C2.1, C4.1, C6.1, R12.1, SW1.2, SW2.2, SW3.2, U6.3 (GND)
- net VCC: now also C2.2, R11.1, U6.1 (VIN)
- new net: C3.1, U6.4 (BST)
- new net: C3.2, L1.1, U6.2 (SW)
- new net: C5.1, R12.2, R13.2, U6.6 (FB)
- new net: R11.2, U6.5 (EN)
Other:
- moved on the sheet: C1, J1, R10, R9, U4

Commit message: AP63203
Parts:
- removed C2: 10u, Capacitor_SMD:C_0603_1608Metric, symbol Device:C
- removed R13: 135k, Resistor_SMD:R_0603_1608Metric, symbol Device:R
- removed U6: PTPS561243DRLR, footprints:DRL0006A-MFG, symbol lib:PTPS561243DRLR
- added C6: 22u, Package_TO_SOT_SMD:TSOT-23-6, symbol Device:C
- added TP1, TP2, TP3, TP4, TP5: TestPoint, Package_SO:TI_SO-PowerPAD-8_ThermalVias, symbol Connector:TestPoint
- added U5: AP63203WU, Package_TO_SOT_SMD:TSOT-23-6, symbol Regulator_Switching:AP63203WU
- C1: renamed from C6; value C -> 0.1u
- C3: value 0.1u -> 100n; footprint Capacitor_SMD:C_0603_1608Metric -> Package_TO_SOT_SMD:TSOT-23-6
- C4: value 22u -> 10u; footprint Capacitor_SMD:C_0603_1608Metric -> Package_TO_SOT_SMD:TSOT-23-6
- C5: value 47p -> 22u; footprint Capacitor_SMD:C_0603_1608Metric -> Package_TO_SOT_SMD:TSOT-23-6
- J1: footprint Package_DFN_QFN:Texas_X2QFN-12_1.6x1.6mm_P0.4mm -> Connector_USB:USB_C_Receptacle_GCT_USB4105-xx-A_16P_TopMnt_Horizontal
- L1: value 1.2u -> 3.9u; footprint (none) -> Inductor_SMD:L_1210_3225Metric
- M1: footprint Package_LCC:PLCC-84_29.3x29.3mm_P1.27mm -> Connector:FanPinHeader_1x04_P2.54mm_Vertical
- R11: value 100k -> 5.1k
- R12: value 30k -> 5.1k
- SW1, SW2, SW3: footprint (none) -> Resistor_THT:R_Axial_DIN0204_L3.6mm_D1.6mm_P5.08mm_Horizontal
- renumbered C1 to C2, R9 to R10, R10 to R9, U2 to U1, U1 to U2, U5 to U4, U4 to U6
Connections:
- net +3V3: now also C6.2, TP2.1, U5.1 (FB); no longer C4.2
- net GND: now also C4.2, C5.1, R11.1, C6.1, TP1.1, U5.4 (GND); no longer C4.1
- net RX: now also TP5.1
- net TX: now also TP4.1
- net UPDI: now also TP3.1
- net at C3.1: now also U5.6 (BST)
- net at C3.2, L1.1: now also U5.5 (SW)
- net at J1.A5 (CC1), U6.4 (CC1): now also R12.2
- net at J1.B5 (CC2), U6.5 (CC2): now also R11.2
- net VCC renamed VBUS
- net VBUS: now also C4.1, U5.2 (EN), U5.3 (IN); no longer R11.1

Commit message: テストポイントとか
Parts:
- removed R12: 5.1k, Resistor_SMD:R_0603_1608Metric, symbol Device:R
- removed TP2: TestPoint, Package_SO:TI_SO-PowerPAD-8_ThermalVias, symbol Connector:TestPoint
- added R10: 5.1k, Resistor_SMD:R_0603_1608Metric, symbol Device:R
- added TP1, TP4, TP5: TestPoint, Package_SO:TI_SO-PowerPAD-8_ThermalVias, symbol Connector:TestPoint
- renumbered R10 to R12, TP1 to TP2, TP4 to TP6, TP5 to TP7
Connections:
- net +3V3: now also TP1.1, TP4.1
- net GND: now also R10.1, TP5.1
- net at J1.A5 (CC1), U6.4 (CC1): now also R10.2
Other:
- moved on the sheet: C2, C3, C4, C5, C6, L1, R12, R9, TP2, TP3, TP6, TP7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

Commit message: OEのPWM
Parts:
- removed TP7: TestPoint, Package_SO:TI_SO-PowerPAD-8_ThermalVias, symbol Connector:TestPoint
Connections:
- net GND: no longer U2.13 (~{OE}), U3.13 (~{OE})
- net PWM: now also U1.8 (PB1); no longer U1.9 (PB0)
- net Tach: now also U1.9 (PB0); no longer U1.8 (PB1)
- net RX renamed 7seg-En
- net 7seg-En: now also U2.13 (~{OE}), U3.13 (~{OE})
Changed lines of the file:
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@@
 		)
 	)
+	(label "Tach"
+		(at 22.86 53.34 180)
+		(effects
+			(font
+				(size 1.27 1.27)
+			)
+			(justify right bottom)
+		)
+	)
 	(label "7seg-3"
 		(at 156.21 63.5 0)
@@
 	)
 	(label "PWM"
-		(at 22.86 53.34 180)
+		(at 22.86 55.88 180)
 		(effects
 			(font
@@
 		)
 	)
+	(label "7seg-En"
+		(at 135.89 68.58 180)
+		(effects
+			(font
+				(size 1.27 1.27)
+			)
+			(justify right bottom)
+		)
+	)
 	(label "TX"
 		(at 22.86 58.42 180)
@@
 		)
 	)
-	(label "RX"
+	(label "7seg-En"
 		(at 22.86 60.96 180)
 		(effects
@@
 		)
 	)
-	(label "Tach"
-		(at 22.86 55.88 180)
-		(effects
-			(font
-				(size 1.27 1.27)
-			)
-			(justify right bottom)
-		)
-	)
 	(label "7seg-C"
 		(at 200.66 60.96 180)
@@
 		)
 	)
-	(label "RX"
-		(at 107.95 26.67 270)
+	(label "7seg-Clock"
+		(at 135.89 58.42 180)
 		(effects
 			(font
@@
 		)
 	)
-	(label "7seg-Clock"
-		(at 135.89 58.42 180)
+	(label "Ctrl-Push"
+		(at 223.52 133.35 180)
 		(effects
 			(font
@@
 		)
 	)
-	(label "Ctrl-Push"
-		(at 223.52 133.35 180)
+	(label "7seg-D"
+		(at 200.66 63.5 180)
 		(effects
 			(font
@@
 		)
 	)
-	(label "7seg-D"
-		(at 200.66 63.5 180)
+	(label "7seg-En"
+		(at 78.74 68.58 180)
 		(effects
 			(font
@@
 	)
 	(symbol
-		(lib_id "Connector:TestPoint")
-		(at 107.95 26.67 0)
-		(unit 1)
-		(body_style 1)
-		(exclude_from_sim no)
-		(in_bom yes)
-		(on_board yes)
-		(in_pos_files yes)
-		(dnp no)
-		(fields_autoplaced yes)
-		(property "Reference" "TP7"
-			(at 110.49 22.0979 0)
-			(show_name no)
-			(do_not_autoplace no)
-			(effects
-				(font
-					(size 1.27 1.27)
-				)
-				(justify left)
-			)
-		)
-		(property "Value" "TestPoint"
-			(at 110.49 24.6379 0)
-			(show_name no)
-			(do_not_autoplace no)
-			(effects
-				(font
-					(size 1.27 1.27)
-				)
-				(justify left)
-			)
-		)
-		(property "Footprint" "Package_SO:TI_SO-PowerPAD-8_ThermalVias"
-			(at 113.03 26.67 0)
-			(hide yes)
-			(show_name no)
-			(do_not_autoplace no)
-			(effects
-				(font
-					(size 1.27 1.27)
-				)
-			)
-		)
-		(property "Datasheet" ""
-			(at 113.03 26.67 0)
-			(hide yes)
-			(show_name no)
-			(do_not_autoplace no)
-			(effects
-				(font
-					(size 1.27 1.27)
-				)
-			)
-		)
-		(property "Description" "test point"
-			(at 107.95 26.67 0)
-			(hide yes)
-			(show_name no)
-			(do_not_autoplace no)
-			(effects
-				(font
-					(size 1.27 1.27)
-				)
-			)
-		)
-		(pin "1"
-		)
-		(instances
-			(project "PCFanController"
-				(path "/52b4d307-cc39-4fe2-86bc-cae0e5ee7f53"
-					(reference "TP7")
-					(unit 1)
-				)
-			)
-		)
-	)
-	(symbol
 		(lib_id "power:GND")
 		(at 177.8 55.88 0)
@@
 	)
 	(symbol
-		(lib_id "power:GND")
-		(at 135.89 68.58 270)
-		(unit 1)
-		(body_style 1)
-		(exclude_from_sim no)
-		(in_bom yes)
-		(on_board yes)
-		(in_pos_files yes)
-		(dnp no)
-		(fields_autoplaced yes)
-		(property "Reference" "#PWR014"
-			(at 129.54 68.58 0)
-			(hide yes)
-			(show_name no)
-			(do_not_autoplace no)
-			(effects
-				(font
-					(size 1.27 1.27)
-				)
-			)
-		)
-		(property "Value" "GND"
-			(at 132.08 68.5799 90)
-			(show_name no)
-			(do_not_autoplace no)
-			(effects
-				(font
-					(size 1.27 1.27)
-				)
-				(justify right)
-			)
-		)
-		(property "Footprint" ""
-			(at 135.89 68.58 0)
-			(hide yes)
-			(show_name no)
-			(do_not_autoplace no)
-			(effects
-				(font
-					(size 1.27 1.27)
-				)
-			)
-		)
-		(property "Datasheet" ""
-			(at 135.89 68.58 0)
-			(hide yes)
-			(show_name no)
-			(do_not_autoplace no)
-			(effects
-				(font
-					(size 1.27 1.27)
-				)
-			)
-		)
-		(property "Description" "Power symbol creates a global label with name \"GND\" , ground"
-			(at 135.89 68.58 0)
-			(hide yes)
-			(show_name no)
-			(do_not_autoplace no)
-			(effects
-				(font
-					(size 1.27 1.27)
-				)
-			)
-		)
-		(pin "1"
-		)
-		(instances
-			(project "PCFanController"
-				(path "/52b4d307-cc39-4fe2-86bc-cae0e5ee7f53"
-					(reference "#PWR014")
-					(unit 1)
-				)
-			)
-		)
-	)
-	(symbol
 		(lib_id "Device:C")
 		(at 80.01 109.22 90)
@@
 					(unit 1)
 				)
-			)
-		)
-	)
-	(symbol
-		(lib_id "power:GND")
-		(at 78.74 68.58 270)
-		(unit 1)
-		(body_style 1)
-		(exclude_from_sim no)
-		(in_bom yes)
-		(on_board yes)
-		(in_pos_files yes)
-		(dnp no)
-		(fields_autoplaced yes)
-		(property "Reference" "#PWR013"
-			(at 72.39 68.58 0)
-			(hide yes)
-			(show_name no)
-			(do_not_autoplace no)
-			(effects
-				(font
-					(size 1.27 1.27)
-				)
-			)
-		)
-		(property "Value" "GND"
-			(at 74.93 68.5799 90)
-			(show_name no)
-			(do_not_autoplace no)
-			(effects
-				(font
-					(size 1.27 1.27)
-				)
-				(justify right)
-			)
-		)
-		(property "Footprint" ""
-			(at 78.74 68.58 0)
-			(hide yes)
-			(show_name no)
-			(do_not_autoplace no)
-			(effects
-				(font
-					(size 1.27 1.27)
-				)
-			)
-		)
-		(property "Datasheet" ""
-			(at 78.74 68.58 0)
-			(hide yes)
-			(show_name no)
-			(do_not_autoplace no)
-			(effects
-				(font
-					(size 1.27 1.27)
-				)
-			)
-		)
-		(property "Description" "Power symbol creates a global label with name \"GND\" , ground"
-			(at 78.74 68.58 0)
-			(hide yes)
-			(show_name no)
-			(do_not_autoplace no)
-			(effects
-				(font
-					(size 1.27 1.27)
-				)
-			)
-		)
-		(pin "1"
-		)
-		(instances
-			(project "PCFanController"
-				(path "/52b4d307-cc39-4fe2-86bc-cae0e5ee7f53"
-					(reference "#PWR013")
-					(unit 1)
-				)

Commit message: ボタン
Parts:
- added C7, C8, C9: C, symbol Device:C
Connections:
- net Ctrl-A: now also C7.1
- net Ctrl-B: now also C8.1
- net Ctrl-Push: now also C9.1
- net GND: now also C7.2, C8.2, C9.2
Other:
- moved on the sheet: SW1, SW3

Commit message: .
Parts:
- C3, C4, C5, C6: footprint Package_TO_SOT_SMD:TSOT-23-6 -> Capacitor_SMD:C_0603_1608Metric
- C7, C8, C9: footprint (none) -> Capacitor_SMD:C_0603_1608Metric
- TP1, TP2, TP3, TP4, TP5, TP6: footprint Package_SO:TI_SO-PowerPAD-8_ThermalVias -> TestPoint:TestPoint_Pad_D1.5mm
Changed lines of the file:
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@@
 			)
 		)
-		(property "Footprint" "Package_SO:TI_SO-PowerPAD-8_ThermalVias"
+		(property "Footprint" "TestPoint:TestPoint_Pad_D1.5mm"
 			(at 30.48 26.67 0)
 			(hide yes)
@@
 			)
 		)
-		(property "Footprint" "Package_SO:TI_SO-PowerPAD-8_ThermalVias"
+		(property "Footprint" "TestPoint:TestPoint_Pad_D1.5mm"
 			(at 100.33 26.67 0)
 			(hide yes)
@@
 			)
 		)
-		(property "Footprint" "Package_SO:TI_SO-PowerPAD-8_ThermalVias"
+		(property "Footprint" "TestPoint:TestPoint_Pad_D1.5mm"
 			(at 74.93 26.67 0)
 			(hide yes)
@@
 			)
 		)
-		(property "Footprint" ""
+		(property "Footprint" "Capacitor_SMD:C_0603_1608Metric"
 			(at 232.41 145.0848 0)
 			(hide yes)
@@
 			)
 		)
-		(property "Footprint" "Package_TO_SOT_SMD:TSOT-23-6"
+		(property "Footprint" "Capacitor_SMD:C_0603_1608Metric"
 			(at 144.78 119.6848 0)
 			(hide yes)
@@
 			)
 		)
-		(property "Footprint" ""
+		(property "Footprint" "Capacitor_SMD:C_0603_1608Metric"
 			(at 232.41 126.0348 0)
 			(hide yes)
@@
 			)
 		)
-		(property "Footprint" "Package_SO:TI_SO-PowerPAD-8_ThermalVias"
+		(property "Footprint" "TestPoint:TestPoint_Pad_D1.5mm"
 			(at 87.63 26.67 0)
 			(hide yes)
@@
 			)
 		)
-		(property "Footprint" "Package_TO_SOT_SMD:TSOT-23-6"
+		(property "Footprint" "Capacitor_SMD:C_0603_1608Metric"
 			(at 151.4348 126.365 0)
 			(hide yes)
@@
 			)
 		)
-		(property "Footprint" "Package_TO_SOT_SMD:TSOT-23-6"
+		(property "Footprint" "Capacitor_SMD:C_0603_1608Metric"
 			(at 115.8748 130.81 0)
 			(hide yes)
@@
 			)
 		)
-		(property "Footprint" "Package_SO:TI_SO-PowerPAD-8_ThermalVias"
+		(property "Footprint" "TestPoint:TestPoint_Pad_D1.5mm"
 			(at 43.18 26.67 0)
 			(hide yes)
@@
 			)
 		)
-		(property "Footprint" "Package_TO_SOT_SMD:TSOT-23-6"
+		(property "Footprint" "Capacitor_SMD:C_0603_1608Metric"
 			(at 145.7452 126.365 0)
 			(hide yes)
@@
 			)
 		)
-		(property "Footprint" "Package_SO:TI_SO-PowerPAD-8_ThermalVias"
+		(property "Footprint" "TestPoint:TestPoint_Pad_D1.5mm"
 			(at 55.88 26.67 0)
 			(hide yes)
@@
 			)
 		)
-		(property "Footprint" ""
+		(property "Footprint" "Capacitor_SMD:C_0603_1608Metric"
 			(at 232.41 106.9848 0)
 			(hide yes)

Commit message: ピンアサイン変更、PCB
Connections:
- net 7seg-A: now also R2.2; no longer R8.2
- net 7seg-B: now also R1.2; no longer R7.2
- net 7seg-C: now also R7.2; no longer R6.2
- net 7seg-G: now also R8.2; no longer R2.2
- net 7seg-P: now also R6.2; no longer R1.2
- net Ctrl-A renamed Button-Disp
- net Button-Disp: now also U1.5 (PA7); no longer U1.3 (PA5)
- net Ctrl-B renamed Button-Plus
- net Ctrl-Push renamed Button-Minus
- net Button-Minus: now also U1.3 (PA5); no longer U1.5 (PA7)

Commit message: テストポイントをスルーホールに変更
Parts:
- removed TP1, TP2, TP3, TP4, TP5, TP6: TestPoint, TestPoint:TestPoint_Pad_D1.5mm, symbol Connector:TestPoint
- added J1, J2: Conn_01x03_Socket, Connector_PinSocket_2.54mm:PinSocket_1x03_P2.54mm_Vertical, symbol Connector:Conn_01x03_Socket
- renumbered C7 to C2, C2 to C3, C3 to C4, C4 to C5, C8 to C6, C5 to C7, C6 to C8, J1 to J3
Connections:
- net +3V3: now also J1.1 (Pin_1), J2.1 (Pin_1)
- net GND: now also J1.2 (Pin_2), J2.2 (Pin_2)
- net TX: now also J2.3 (Pin_3)
- net UPDI: now also J1.3 (Pin_3)
