File: PCB/PCFanController.kicad_pcb (KiCad board)
At the start: 2 copper layers, 65.5 x 30 mm, 37 parts, among them J1 Conn_01x03_Socket, J2 Conn_01x03_Socket, J3 USB_C_Receptacle_USB2.0_16P, M1 Fan_4pin, Q1 BSS138, Q2 MTN2306AN3, SW1 SW_Push, SW2 SW_Push, SW3 SW_Push, U1 ATtiny404-SS, U2 74HC595, U3 74HC595, U4 OSL40562-LR, U5 AP63203WU, U6 CH221K

Commit message: びあ
Parts:
- moved C4 0.50 mm to (108.5, 85.5)
- moved M1 0.50 mm to (76.2, 83.2)
Routing:
- net +3V3: track 44.6 -> 37.9 mm, vias 9 -> 8
- net /Fan-Gnd: track 5.73 -> 5.23 mm
- net GND: vias 65 -> 68
Other:
- board text added: "0.1u ATtiny404 BSS138"
- board text added: "10u AP63203 2x22u 3.9u 100n"
- board text added: "1u 1k CH221K 47k"
- board text added: "3xNC 3xSKRG"
- board text added: "8xR_LED"
- board text added: "MTN2306"
- board text added: "USB-C 2x5.1k"
- board text added: "l.dg7.dev/fan"

Commit message: 抵抗値変更
Parts:
- R1, R2, R3, R4, R5, R6, R7, R8: value 330 -> 180
Changed lines of the file:
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@@
 			)
 		)
-		(property "Value" "330"
+		(property "Value" "180"
 			(at 0 1.43 90)
 			(layer "F.Fab")
@@
 			)
 		)
-		(property "Value" "330"
+		(property "Value" "180"
 			(at 0 1.43 90)
 			(layer "F.Fab")
@@
 			)
 		)
-		(property "Value" "330"
+		(property "Value" "180"
 			(at 0 1.43 90)
 			(layer "F.Fab")
@@
 			)
 		)
-		(property "Value" "330"
+		(property "Value" "180"
 			(at 0 1.43 90)
 			(layer "F.Fab")
@@
 			)
 		)
-		(property "Value" "330"
+		(property "Value" "180"
 			(at 0 1.43 90)
 			(layer "F.Fab")
@@
 			)
 		)
-		(property "Value" "330"
+		(property "Value" "180"
 			(at 0 1.43 0)
 			(layer "F.Fab")
@@
 			)
 		)
-		(property "Value" "330"
+		(property "Value" "180"
 			(at 0 1.43 90)
 			(layer "F.Fab")
@@
 			)
 		)
-		(property "Value" "330"
+		(property "Value" "180"
 			(at 0 1.43 90)
 			(layer "F.Fab")

Commit message: 銅箔
Other:
- board text added: "2x74HC595"
- board text added: "OSL40562"
Changed lines of the file:
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@@
 		(layer "Edge.Cuts")
+	)
+	(gr_text "UG3\nTG3"
+		(at 125.5 82 0)
+		(layer "F.Mask")
+		(effects
+			(font
+				(size 0.8 0.8)
+				(thickness 0.16)
+				(bold yes)
+			)
+		)
+	)
+	(gr_text "DISP"
+		(at 138 88 0)
+		(layer "F.Mask")
+		(effects
+			(font
+				(size 0.8 0.8)
+				(thickness 0.16)
+				(bold yes)
+			)
+		)
+	)
+	(gr_text "+"
+		(at 138 98 0)
+		(layer "F.Mask")
+		(effects
+			(font
+				(size 0.8 0.8)
+				(thickness 0.16)
+				(bold yes)
+			)
+		)
+	)
+	(gr_text "-\n"
+		(at 138 102 0)
+		(layer "F.Mask")
+		(effects
+			(font
+				(size 0.8 0.8)
+				(thickness 0.16)
+				(bold yes)
+			)
+		)
+	)
+	(gr_text "l.dg7.dev/fan"
+		(at 139 108.5 0)
+		(layer "F.Mask")
+		(effects
+			(font
+				(size 0.8 0.8)
+				(thickness 0.16)
+				(bold yes)
+			)
+			(justify right)
+		)
 	)
 	(gr_text "MTN2306\n"
@@
 		)
 	)
+	(gr_text "OSL40562"
+		(at 92.5 94 0)
+		(layer "F.SilkS")
+		(effects
+			(font
+				(size 0.8 0.8)
+				(thickness 0.16)
+				(bold yes)
+			)
+			(justify left)
+		)
+	)
 	(gr_text "8xR_LED"
 		(at 97 95.5 0)
+		(layer "F.SilkS")
+		(effects
+			(font
+				(size 0.8 0.8)
+				(thickness 0.16)
+				(bold yes)
+			)
+			(justify left)
+		)
+	)
+	(gr_text "2x74HC595"
+		(at 109.5 92.5 0)
 		(layer "F.SilkS")
 		(effects
@@
 		)
 	)
-	(gr_text "UG3\nTG3"
-		(at 125.5 82 0)
-		(layer "F.SilkS")
-		(effects
-			(font
-				(size 0.8 0.8)
-				(thickness 0.16)
-				(bold yes)
-			)
-		)
-	)
-	(gr_text "DISP"
-		(at 138 88 0)
-		(layer "F.SilkS")
-		(effects
-			(font
-				(size 0.8 0.8)
-				(thickness 0.16)
-				(bold yes)
-			)
-		)
-	)
-	(gr_text "+"
-		(at 138 98 0)
-		(layer "F.SilkS")
-		(effects
-			(font
-				(size 0.8 0.8)
-				(thickness 0.16)
-				(bold yes)
-			)
-		)
-	)
-	(gr_text "-\n"
-		(at 138 102 0)
-		(layer "F.SilkS")
-		(effects
-			(font
-				(size 0.8 0.8)
-				(thickness 0.16)
-				(bold yes)
-			)
-		)
-	)
-	(gr_text "l.dg7.dev/fan"
-		(at 139.5 109 0)
-		(layer "F.SilkS")
-		(effects
-			(font
-				(size 0.8 0.8)
-				(thickness 0.16)
-				(bold yes)
-			)
-			(justify right)
-		)
-	)
