File: PCB/PCFanController.kicad_pcb (KiCad board)
At the start: 2 copper layers, 65.5 x 30 mm, 37 parts, among them J1 Conn_01x03_Socket, J2 Conn_01x03_Socket, J3 USB_C_Receptacle_USB2.0_16P, M1 Fan_4pin, Q1 BSS138, Q2 MTN2306AN3, SW1 SW_Push, SW2 SW_Push, SW3 SW_Push, U1 ATtiny404-SS, U2 74HC595, U3 74HC595, U4 OSL40562-LR, U5 AP63203WU, U6 CH221K

Commit message: ファンのピンアサイン
Other:
- board text added: "GVTP"
- board text removed: "G"
Changed lines of the file:
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@@
 		(layer "Edge.Cuts")
+	)
+	(gr_text "GVTP"
+		(at 77 81.5 0)
+		(layer "F.Mask")
+		(effects
+			(font
+				(size 0.8 0.8)
+				(thickness 0.16)
+				(bold yes)
+			)
+			(justify left)
+		)
 	)
 	(gr_text "UG3\nTG3"
@@
 		)
 	)
-	(gr_text "G"
-		(at 76 81.5 0)
-		(layer "F.SilkS")
-		(effects
-			(font
-				(size 0.8 0.8)
-				(thickness 0.16)
-				(bold yes)
-			)
-		)
-	)
